Commit message: Day 6: LiDAR 센서 설정 변경 - 360도 스캔, 중앙 배치, 높이 조정, laser_filters 적용

File: src/mastering_ros_robot_description_pkg/urdf/diff_wheeled_robot_with_laser.xacro (robot description, xacro)
@@ -42,4 +42,5 @@
   <!-- Hokuyo Laser scanner -->
   <xacro:property name="hokuyo_size" value="0.05" />
+  <xacro:property name="laser_height" value="0.08" />
   <!-- Macro for calculating inertia of cylinder -->
   <xacro:macro name="cylinder_inertia" params="m r h">
@@ -195,5 +196,5 @@
   </link>
   <joint name="hokuyo_joint" type="fixed">
-    <origin xyz="${base_radius - hokuyo_size/2} 0 ${base_height+hokuyo_size/4}" rpy="0 0 0" />
+    <origin xyz="0 0 ${base_height+hokuyo_size/4}" rpy="0 0 0" />
     <parent link="base_link"/>
     <child link="laser_link" />
@@ -211,6 +212,6 @@
             <samples>720</samples>
             <resolution>1</resolution>
-            <min_angle>-1.570796</min_angle>
-            <max_angle>1.570796</max_angle>
+            <min_angle>-3.141593</min_angle>
+            <max_angle>3.141593</max_angle>
           </horizontal>
         </scan>
